File: PCB/opengbc-pcb/audio.kicad_sch (KiCad schematic)
At the start: 0 parts

Commit message: update audio schematic
Parts:
- added C2, C3, C4: 1uF, symbol Device:C_Small
- added C5, C6: 100uF, symbol Device:C_Small
- added P5: AudioJack3_Switch, symbol Connector_Audio:AudioJack3_Switch
- added R1, R2: 510, symbol Device:R_US
- added R3, R4, R6: 100k, symbol Device:R_US
- added R5, R7: 1k, symbol Device:R_US
- added R8, R9: 20k, symbol Device:R_US
- added RV1: 10k x2, symbol Device:R_Potentiometer_Dual
- added SP1: Speaker, symbol Device:Speaker
- added U3: LM4853, SOP50P490X110-10N, symbol LM4853MM_NOPB:LM4853MM_NOPB
Connections:
- new net: R3.2, R8.1, U3.1 (LEFT_IN)
- new net: C5.1, R8.2, SP1.2, U3.10 (LEFT_OUT/BTL_OUT-)
- new net: P5.RN, R6.2, U3.3 (HP-IN)
- new net: R4.2, R9.2, U3.5 (RIGHT_IN)
- new net: C6.1, R9.1, U3.6 (RIGHT_OUT)
- new net: C4.1, U3.7 (BYPASS)
- new net: SP1.1, U3.8 (BTL_OUT+)
- new net: C3.2, R2.1
- new net: R2.2, RV1.4
- new net: C6.2, P5.R, R7.1
- new net: C5.2, P5.T, R5.1
- new net: R3.1, RV1.2
- new net: C2.2, R1.1
- new net: R1.2, RV1.1
- new net: R4.1, RV1.5
- new net +5V: R6.1, U3.9 (VDD)
- new net GND: C4.2, P5.S, R5.2, R7.2, RV1.3, RV1.6, U3.2 (SHUTDOWN), U3.4 (GND)
- new net S01: C3.1
- new net S02: C2.1
- no-connect marks 0 -> 2

Commit message: :eyes:
Parts:
- C2, C3, C4: footprint (none) -> Capacitor_SMD:C_0603_1608Metric_Pad1.08x0.95mm_HandSolder; Mouser Part Number (none) -> 963-JMK107BJ105MA-T
- C5, C6: footprint (none) -> Capacitor_SMD:C_1206_3216Metric_Pad1.33x1.80mm_HandSolder; Mouser Part Number (none) -> 187-CL31A107MQHNNWE
- P5: footprint (none) -> gbc_repro_lib:audio_jack; symbol Connector_Audio:AudioJack3_Switch -> Connector_Audio:AudioJack3_SwitchTR; Mouser Part Number (none) -> 490-SJ1-3525N
- R1, R2: value 510 -> 510R; footprint (none) -> Resistor_SMD:R_0603_1608Metric_Pad0.98x0.95mm_HandSolder; Mouser Part Number (none) -> 791-WR06X511JTL
- R3, R4, R6: footprint (none) -> Resistor_SMD:R_0603_1608Metric_Pad0.98x0.95mm_HandSolder; Mouser Part Number (none) -> 279-CRGCQ0603F100K
- R5, R7: footprint (none) -> Resistor_SMD:R_0603_1608Metric_Pad0.98x0.95mm_HandSolder; Mouser Part Number (none) -> 603-AC0603JR-131KL
- R8, R9: footprint (none) -> Resistor_SMD:R_0603_1608Metric_Pad0.98x0.95mm_HandSolder; Mouser Part Number (none) -> 660-RN73R1JTD2002F25
- RV1: footprint (none) -> gbc_repro_lib:gbc_volume_wheel; symbol Device:R_Potentiometer_Dual -> gbc_volume:R_Potentiometer_Dual; Mouser Part Number (none) -> 688-RK10J12R0A0B
- SP1: footprint (none) -> Connector_PinHeader_1.00mm:PinHeader_1x02_P1.00mm_Vertical; now left out of the parts list
- U3: footprint SOP50P490X110-10N -> Package_SO:VSSOP-10_3x3mm_P0.5mm
Connections:
- net GND: now also RV1.1 (GND); no longer RV1.3, RV1.6
- net at R2.2: now also RV1.5 (S01_IN); no longer RV1.4
- net at R3.1: now also RV1.3 (S02_OUT); no longer RV1.2
- net at R1.2: now also RV1.4 (S02_IN); no longer RV1.1
- net at R4.1: now also RV1.2 (S02_OUT); no longer RV1.5
- no-connect marks 2 -> 1
Changed lines of the file:
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@@
-	)
-	(no_connect
-		(at 209.55 83.82)
 	)
 	(no_connect
@@
 			)
 		)
-		(property "Footprint" "SOP50P490X110-10N"
+		(property "Footprint" "Package_SO:VSSOP-10_3x3mm_P0.5mm"
 			(at 176.53 166.04 0)
 			(effects
@@
 			)
 		)
-		(property "Value" "510"
+		(property "Value" "510R"
 			(at 69.85 78.74 90)
 			(effects
@@
 			)
 		)
-		(property "Footprint" ""
+		(property "Footprint" "Resistor_SMD:R_0603_1608Metric_Pad0.98x0.95mm_HandSolder"
 			(at 70.104 81.534 90)
 			(effects
@@
 		(property "Description" "Resistor, US symbol"
 			(at 69.85 82.55 0)
+			(effects
+				(font
+					(size 1.27 1.27)
+				)
+				(hide yes)
+			)
+		)
+		(property "Mouser Part Number" " 791-WR06X511JTL "
+			(at 69.85 82.55 90)
 			(effects
 				(font
@@
 			)
 		)
-		(property "Footprint" ""
+		(property "Footprint" "Capacitor_SMD:C_0603_1608Metric_Pad1.08x0.95mm_HandSolder"
 			(at 59.69 82.55 0)
 			(effects
@@
 			)
 		)
+		(property "Mouser Part Number" " 963-JMK107BJ105MA-T "
+			(at 59.69 82.55 90)
+			(effects
+				(font
+					(size 1.27 1.27)
+				)
+				(hide yes)
+			)
+		)
 		(pin "2"
 		)
@@
 	)
 	(symbol
-		(lib_id "Connector_Audio:AudioJack3_Switch")
+		(lib_id "Connector_Audio:AudioJack3_SwitchTR")
 		(at 214.63 81.28 180)
 		(unit 1)
@@
 		(fields_autoplaced yes)
 		(property "Reference" "P5"
-			(at 222.25 78.7399 0)
+			(at 222.25 76.8349 0)
 			(effects
 				(font
@@
 		)
 		(property "Value" "AudioJack3_Switch"
-			(at 222.25 81.2799 0)
+			(at 222.25 79.3749 0)
 			(effects
 				(font
@@
 			)
 		)
-		(property "Footprint" ""
+		(property "Footprint" "gbc_repro_lib:audio_jack"
 			(at 214.63 81.28 0)
 			(effects
@@
 			)
 		)
-		(property "Description" "Audio Jack, 3 Poles (Stereo / TRS), Switched Poles (Normalling)"
+		(property "Description" "Audio Jack, 3 Poles (Stereo / TRS), Switched TR Poles (Normalling)"
 			(at 214.63 81.28 0)
 			(effects
@@
 			)
 		)
-		(pin "SN"
+		(property "Mouser Part Number" " 490-SJ1-3525N "
+			(at 214.63 81.28 0)
+			(effects
+				(font
+					(size 1.27 1.27)
+				)
+				(hide yes)
+			)
 		)
 		(pin "S"
@@
 			)
 		)
-		(property "Footprint" ""
+		(property "Footprint" "Capacitor_SMD:C_1206_3216Metric_Pad1.33x1.80mm_HandSolder"
 			(at 185.42 78.74 0)
 			(effects
@@
 		(property "Description" "Unpolarized capacitor, small symbol"
 			(at 185.42 78.74 0)
+			(effects
+				(font
+					(size 1.27 1.27)
+				)
+				(hide yes)
+			)
+		)
+		(property "Mouser Part Number" "187-CL31A107MQHNNWE"
+			(at 185.42 78.74 90)
 			(effects
 				(font
@@
 			)
 		)
-		(property "Footprint" ""
+		(property "Footprint" "Resistor_SMD:R_0603_1608Metric_Pad0.98x0.95mm_HandSolder"
 			(at 113.284 61.976 90)
 			(effects
@@
 		)
 		(property "Description" "Resistor, US symbol"
+			(at 114.3 62.23 0)
+			(effects
+				(font
+					(size 1.27 1.27)
+				)
+				(hide yes)
+			)
+		)
+		(property "Mouser Part Number" " 660-RN73R1JTD2002F25 "
 			(at 114.3 62.23 0)
 			(effects
@@
 			)
 		)
-		(property "Footprint" ""
+		(property "Footprint" "Resistor_SMD:R_0603_1608Metric_Pad0.98x0.95mm_HandSolder"
 			(at 103.124 72.644 90)
 			(effects
@@
 			)
 		)
+		(property "Mouser Part Number" " 279-CRGCQ0603F100K "
+			(at 102.87 73.66 90)
+			(effects
+				(font
+					(size 1.27 1.27)
+				)
+				(hide yes)
+			)
+		)
 		(pin "1"
 		)
@@
 			)
 		)
-		(property "Footprint" ""
+		(property "Footprint" "Capacitor_SMD:C_1206_3216Metric_Pad1.33x1.80mm_HandSolder"
 			(at 185.42 99.06 0)
 			(effects
@@
 		(property "Description" "Unpolarized capacitor, small symbol"
 			(at 185.42 99.06 0)
+			(effects
+				(font
+					(size 1.27 1.27)
+				)
+				(hide yes)
+			)
+		)
+		(property "Mouser Part Number" "187-CL31A107MQHNNWE"
+			(at 185.42 99.06 90)
 			(effects
 				(font
@@
 			)
 		)
-		(property "Value" "510"
+		(property "Value" "510R"
 			(at 69.85 66.04 90)
 			(effects
@@
 			)
 		)
-		(property "Footprint" ""
+		(property "Footprint" "Resistor_SMD:R_0603_1608Metric_Pad0.98x0.95mm_HandSolder"
 			(at 70.104 68.834 90)
 			(effects
@@
 			)
 		)
+		(property "Mouser Part Number" " 791-WR06X511JTL "
+			(at 69.85 69.85 90)
+			(effects
+				(font
+					(size 1.27 1.27)
+				)
+				(hide yes)
+			)
+		)
 		(pin "2"
 		)
@@
 		(unit 1)
 		(exclude_from_sim no)
-		(in_bom yes)
+		(in_bom no)
 		(on_board yes)
 		(dnp no)
@@
 			)
 		)
-		(property "Footprint" ""
+		(property "Footprint" "Connector_PinHeader_1.00mm:PinHeader_1x02_P1.00mm_Vertical"
 			(at 172.72 62.23 0)
 			(effects
@@
 		(property "Description" "Speaker"
 			(at 167.64 62.23 0)
+			(effects
+				(font
+					(size 1.27 1.27)
+				)
+				(hide yes)
+			)
+		)
+		(property "Mouser Part Number" "~"
+			(at 167.64 62.23 90)
 			(effects
 				(font
@@
 			)
 		)
-		(property "Footprint" ""
+		(property "Footprint" "Resistor_SMD:R_0603_1608Metric_Pad0.98x0.95mm_HandSolder"
 			(at 194.056 103.124 90)
 			(effects
@@
 			)
 		)
+		(property "Mouser Part Number" " 603-AC0603JR-131KL "
+			(at 193.04 102.87 0)
+			(effects
+				(font
+					(size 1.27 1.27)
+				)
+				(hide yes)
+			)
+		)
 		(pin "2"
 		)
@@
 	)
 	(symbol
-		(lib_id "Device:R_Potentiometer_Dual")
+		(lib_id "gbc_volume:R_Potentiometer_Dual")
 		(at 85.09 80.01 270)
 		(unit 1)
@@
 			)
 		)
-		(property "Footprint" ""
+		(property "Footprint" "gbc_repro_lib:gbc_volume_wheel"
 			(at 83.185 86.36 0)
 			(effects
@@
 			)
 		)
-		(pin "6"
+		(property "Mouser Part Number" " 688-RK10J12R0A0B "
+			(at 85.09 80.01 90)
+			(effects
+				(font
+					(size 1.27 1.27)
+				)
+				(hide yes)
+			)
+		)
+		(pin "1"
 		)
 		(pin "2"
@@
 			)
 		)
-		(property "Footprint" ""
+		(property "Footprint" "Resistor_SMD:R_0603_1608Metric_Pad0.98x0.95mm_HandSolder"
 			(at 175.006 91.694 90)
 			(effects
@@
 		)
 		(property "Description" "Resistor, US symbol"
+			(at 173.99 91.44 0)
+			(effects
+				(font
+					(size 1.27 1.27)
+				)
+				(hide yes)
+			)
+		)
+		(property "Mouser Part Number" " 279-CRGCQ0603F100K "
 			(at 173.99 91.44 0)
 			(effects
@@
 			)
 		)
-		(property "Footprint" ""
+		(property "Footprint" "Resistor_SMD:R_0603_1608Metric_Pad0.98x0.95mm_HandSolder"
 			(at 113.284 112.776 90)
 			(effects
@@
 		)
 		(property "Description" "Resistor, US symbol"
+			(at 114.3 113.03 0)
+			(effects
+				(font
+					(size 1.27 1.27)
+				)
+				(hide yes)
+			)
+		)
+		(property "Mouser Part Number" " 660-RN73R1JTD2002F25 "
 			(at 114.3 113.03 0)
 			(effects
@@
 			)
 		)
-		(property "Footprint" ""
+		(property "Footprint" "Resistor_SMD:R_0603_1608Metric_Pad0.98x0.95mm_HandSolder"
 			(at 194.056 82.804 90)
 			(effects
@@
 		)
 		(property "Description" "Resistor, US symbol"
+			(at 193.04 82.55 0)
+			(effects
+				(font
+					(size 1.27 1.27)
+				)
+				(hide yes)
+			)
+		)
+		(property "Mouser Part Number" " 603-AC0603JR-131KL "
 			(at 193.04 82.55 0)
 			(effects
@@
 			)
 		)
-		(property "Footprint" ""
+		(property "Footprint" "Resistor_SMD:R_0603_1608Metric_Pad0.98x0.95mm_HandSolder"
 			(at 103.124 85.344 90)
 			(effects
@@
 		(property "Description" "Resistor, US symbol"
 			(at 102.87 86.36 0)
+			(effects
+				(font
+					(size 1.27 1.27)
+				)
+				(hide yes)
+			)
+		)
+		(property "Mouser Part Number" " 279-CRGCQ0603F100K "
+			(at 102.87 86.36 90)
 			(effects
 				(font
@@
 	(symbol
 		(lib_id "power:GND")
-		(at 209.55 86.36 0)
+		(at 209.55 83.82 0)
 		(unit 1)
 		(exclude_from_sim no)
@@
 		(fields_autoplaced yes)
 		(property "Reference" "#PWR029"
-			(at 209.55 92.71 0)
+			(at 209.55 90.17 0)
 			(effects
 				(font
@@
 		)
 		(property "Value" "GND"
-			(at 209.55 91.44 0)
+			(at 209.55 88.9 0)
 			(effects
 				(font
@@
 		)
 		(property "Footprint" ""
-			(at 209.55 86.36 0)
+			(at 209.55 83.82 0)
 			(effects
 				(font
@@
 		)
 		(property "Datasheet" ""
-			(at 209.55 86.36 0)
+			(at 209.55 83.82 0)
 			(effects
 				(font
@@
 		)
 		(property "Description" "Power symbol creates a global label with name \"GND\" , ground"
-			(at 209.55 86.36 0)
+			(at 209.55 83.82 0)
 			(effects
 				(font
@@
 			)
 		)
-		(property "Footprint" ""
+		(property "Footprint" "Capacitor_SMD:C_0603_1608Metric_Pad1.08x0.95mm_HandSolder"
 			(at 59.69 69.85 0)
 			(effects
@@
 		(property "Description" "Unpolarized capacitor, small symbol"
 			(at 59.69 69.85 0)
+			(effects
+				(font
+					(size 1.27 1.27)
+				)
+				(hide yes)
+			)
+		)
+		(property "Mouser Part Number" " 963-JMK107BJ105MA-T "
+			(at 59.69 69.85 90)
 			(effects
 				(font
@@
 			)
 		)
-		(property "Footprint" ""
+		(property "Footprint" "Capacitor_SMD:C_0603_1608Metric_Pad1.08x0.95mm_HandSolder"
 			(at 120.65 95.25 0)
 			(effects
@@
 			(at 120.65 95.25 0)
 			(effects
+				(font
+					(size 1.27 1.27)
+				)
+				(hide yes)
+			)
+		)
+		(property "Mouser Part Number" " 963-JMK107BJ105MA-T "
+			(at 120.65 95.25 0)
+			(effects
