File: PCB/opengbc-pcb/disp_ffc.kicad_sch (KiCad schematic)
At the start: 2 parts, among them P2 DISP_FFC

Commit message: whole bunch of schematic updates
Connections:
- net at P2.10 (VEE): no longer P2.9 (VEE)
- net at P2.11 (VCOM): no longer P2.12 (VCOM)
- no-connect marks 13 -> 17
Changed lines of the file:
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@@
+	)
+	(no_connect
+		(at 154.94 146.05)
 	)
 	(no_connect
@@
 	)
 	(no_connect
+		(at 154.94 140.97)
+	)
+	(no_connect
 		(at 154.94 167.64)
 	)
 	(no_connect
 		(at 154.94 48.26)
+	)
+	(no_connect
+		(at 154.94 143.51)
 	)
 	(no_connect
@@
 	(no_connect
 		(at 154.94 35.56)
+	)
+	(no_connect
+		(at 154.94 138.43)
 	)
 	(no_connect
@@
 	(wire
 		(pts
-			(xy 154.94 140.97) (xy 154.94 138.43)
-		)
-		(stroke
-			(width 0)
-			(type default)
-		)
-	)
-	(wire
-		(pts
 			(xy 148.59 80.01) (xy 154.94 80.01)
 		)
@@
 		)
 		(stroke
-			(width 0)
-			(type default)
-		)
-	)
-	(wire
-		(pts
-			(xy 154.94 146.05) (xy 154.94 143.51)
-		)
-		(stroke

Commit message: :eyes:
Parts:
- C1: footprint (none) -> Capacitor_SMD:C_0603_1608Metric_Pad1.08x0.95mm_HandSolder; Mouser Part Number (none) -> 81-GRM033R61C104KE4D
- P2: footprint (none) -> gbc_repro_lib:AMPHENOL_62684-502100AHLF; Mouser Part Number (none) -> 649-62684-502100AHLF
Connections:
- net GND: now also P2.SH (Shield)
Changed lines of the file:
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@@
 			)
 		)
-		(property "Footprint" ""
+		(property "Footprint" "Capacitor_SMD:C_0603_1608Metric_Pad1.08x0.95mm_HandSolder"
 			(at 139.3952 54.61 0)
 			(effects
@@
 		)
 		(property "Description" "Unpolarized capacitor"
+			(at 138.43 50.8 0)
+			(effects
+				(font
+					(size 1.27 1.27)
+				)
+				(hide yes)
+			)
+		)
+		(property "Mouser Part Number" " 81-GRM033R61C104KE4D "
 			(at 138.43 50.8 0)
 			(effects
@@
 	)
 	(symbol
+		(lib_id "power:GND")
+		(at 162.56 191.77 0)
+		(unit 1)
+		(exclude_from_sim no)
+		(in_bom yes)
+		(on_board yes)
+		(dnp no)
+		(fields_autoplaced yes)
+		(property "Reference" "#PWR069"
+			(at 162.56 198.12 0)
+			(effects
+				(font
+					(size 1.27 1.27)
+				)
+				(hide yes)
+			)
+		)
+		(property "Value" "GND"
+			(at 162.56 196.85 0)
+			(effects
+				(font
+					(size 1.27 1.27)
+				)
+			)
+		)
+		(property "Footprint" ""
+			(at 162.56 191.77 0)
+			(effects
+				(font
+					(size 1.27 1.27)
+				)
+				(hide yes)
+			)
+		)
+		(property "Datasheet" ""
+			(at 162.56 191.77 0)
+			(effects
+				(font
+					(size 1.27 1.27)
+				)
+				(hide yes)
+			)
+		)
+		(property "Description" "Power symbol creates a global label with name \"GND\" , ground"
+			(at 162.56 191.77 0)
+			(effects
+				(font
+					(size 1.27 1.27)
+				)
+				(hide yes)
+			)
+		)
+		(pin "1"
+		)
+		(instances
+			(project ""
+				(path "/3a870878-1e85-4537-97d1-09e5db9009a0/c4a329d8-d5ce-4d4d-ae4b-d07fca2cf265"
+					(reference "#PWR069")
+					(unit 1)
+				)
+			)
+		)
+	)
+	(symbol
 		(lib_id "gbc_display:DISP_FFC")
 		(at 162.56 66.04 0)
@@
 			)
 		)
-		(property "Footprint" ""
+		(property "Footprint" "gbc_repro_lib:AMPHENOL_62684-502100AHLF"
 			(at 162.56 66.04 0)
 			(effects
@@
 			)
 		)
+		(property "Mouser Part Number" " 649-62684-502100AHLF "
+			(at 162.56 66.04 0)
+			(effects
+				(font
+					(size 1.27 1.27)
+				)
+				(hide yes)
+			)
+		)
 		(pin "40"
 		)
@@
 		(pin "30"
 		)
-		(instances
+		(pin "SH"
+		)
+		(instances
