File: PCB/opengbc-pcb/ir.kicad_sch (KiCad schematic)
At the start: 0 parts

Commit message: whole bunch of schematic updates
Parts:
- added C12: .47uF, symbol Device:C
- added C13: 33pF, symbol Device:C
- added C14: .015uF, symbol Device:C_Small
- added C15: 1uF, symbol Device:C
- added D1: IR LED, symbol Device:LED
- added Q1, Q2: 2SC4081UB, symbol Transistor_BJT:Q_NPN_BEC
- added Q3: PT380F, symbol Device:Q_Photo_NPN_EC
- added R10: 1k, symbol Device:R_US
- added R11: 150R, symbol Device:R_US
- added R12: 200k, symbol Device:R_US
- added R13: 4.7k, symbol Device:R_US
- added R14: 1M, symbol Device:R_US
- added R15: 2k, symbol Device:R_US
- added R16, R17: 33k, symbol Device:R_US
Connections:
- new net: C15.1, Q2.1 (B), R16.2, R17.1
- new net: Q2.2 (E), Q3.2 (C)
- new net: C14.1, Q2.3 (C), R15.2
- new net: C14.2, R13.1, R14.2
- new net: D1.1 (K), Q1.3 (C)
- new net: D1.2 (A), R10.1, R11.2
- new net: C12.1, R10.2
- new net +5V: R11.1
- new net GND: C12.2, C15.2, Q1.2 (E), Q3.1 (E), R17.2
- new net R0: Q1.1 (B)
- new net R1: R14.1, R15.1, R16.1
- new net R2: C13.1, R12.1, R13.2
- new net R3: C13.2, R12.2

Commit message: :eyes:
Parts:
- C12: footprint (none) -> Capacitor_SMD:C_0603_1608Metric_Pad1.08x0.95mm_HandSolder; Mouser Part Number (none) -> 810-CGA3E2X5R1A474MA
- C13: footprint (none) -> Capacitor_SMD:C_0603_1608Metric_Pad1.08x0.95mm_HandSolder; Mouser Part Number (none) -> 187-CL10C330JB8NNND
- C14: footprint (none) -> Capacitor_SMD:C_0603_1608Metric_Pad1.08x0.95mm_HandSolder; Mouser Part Number (none) -> 80-C0603C153K4RECTU
- C15: footprint (none) -> Capacitor_SMD:C_0603_1608Metric_Pad1.08x0.95mm_HandSolder; Mouser Part Number (none) -> 963-JMK107BJ105MA-T
- D1, Q3: footprint (none) -> gbc_repro_lib:gbc_ir_leds; now left out of the parts list
- Q1, Q2: footprint (none) -> Package_TO_SOT_SMD:SOT-323_SC-70; Mouser Part Number (none) -> 755-2SC4081UBTLR
- R10: footprint (none) -> Resistor_SMD:R_0603_1608Metric_Pad0.98x0.95mm_HandSolder; Mouser Part Number (none) -> 603-AC0603JR-131KL
- R11: footprint (none) -> Resistor_SMD:R_0603_1608Metric_Pad0.98x0.95mm_HandSolder; Mouser Part Number (none) -> 708-RMCF0603JT150R
- R12: footprint (none) -> Resistor_SMD:R_0603_1608Metric_Pad0.98x0.95mm_HandSolder; Mouser Part Number (none) -> 603-AC0603JR-07200KL
- R13: footprint (none) -> Resistor_SMD:R_0603_1608Metric_Pad0.98x0.95mm_HandSolder; Mouser Part Number (none) -> 791-RMC16-472JTP
- R14: footprint (none) -> Resistor_SMD:R_0603_1608Metric_Pad0.98x0.95mm_HandSolder; Mouser Part Number (none) -> 279-CRG0603F1M0
- R15: footprint (none) -> Resistor_SMD:R_0603_1608Metric_Pad0.98x0.95mm_HandSolder; Mouser Part Number (none) -> 603-RT0603DRE072KL
- R16, R17: footprint (none) -> Resistor_SMD:R_0603_1608Metric_Pad0.98x0.95mm_HandSolder; Mouser Part Number (none) -> 791-WR06X333JTL
Changed lines of the file:
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@@
 			)
 		)
-		(property "Footprint" ""
+		(property "Footprint" "Package_TO_SOT_SMD:SOT-323_SC-70"
 			(at 106.68 96.52 0)
 			(effects
@@
 		)
 		(property "Description" "NPN transistor, base/emitter/collector"
+			(at 101.6 99.06 0)
+			(effects
+				(font
+					(size 1.27 1.27)
+				)
+				(hide yes)
+			)
+		)
+		(property "Mouser Part Number" " 755-2SC4081UBTLR "
 			(at 101.6 99.06 0)
 			(effects
@@
 			)
 		)
-		(property "Footprint" ""
+		(property "Footprint" "Resistor_SMD:R_0603_1608Metric_Pad0.98x0.95mm_HandSolder"
 			(at 129.286 98.044 90)
 			(effects
@@
 		)
 		(property "Description" "Resistor, US symbol"
+			(at 128.27 97.79 0)
+			(effects
+				(font
+					(size 1.27 1.27)
+				)
+				(hide yes)
+			)
+		)
+		(property "Mouser Part Number" " 791-RMC16-472JTP "
 			(at 128.27 97.79 0)
 			(effects
@@
 			)
 		)
-		(property "Footprint" ""
+		(property "Footprint" "Capacitor_SMD:C_0603_1608Metric_Pad1.08x0.95mm_HandSolder"
 			(at 75.8952 106.68 0)
 			(effects
@@
 		)
 		(property "Description" "Unpolarized capacitor"
+			(at 74.93 102.87 0)
+			(effects
+				(font
+					(size 1.27 1.27)
+				)
+				(hide yes)
+			)
+		)
+		(property "Mouser Part Number" " 963-JMK107BJ105MA-T "
 			(at 74.93 102.87 0)
 			(effects
@@
 			)
 		)
-		(property "Footprint" ""
+		(property "Footprint" "Package_TO_SOT_SMD:SOT-323_SC-70"
 			(at 130.81 50.8 0)
 			(effects
@@
 			)
 		)
+		(property "Mouser Part Number" " 755-2SC4081UBTLR "
+			(at 135.89 53.34 0)
+			(effects
+				(font
+					(size 1.27 1.27)
+				)
+				(hide yes)
+			)
+		)
 		(pin "2"
 		)
@@
 			)
 		)
-		(property "Footprint" ""
+		(property "Footprint" "Capacitor_SMD:C_0603_1608Metric_Pad1.08x0.95mm_HandSolder"
 			(at 116.84 93.98 0)
 			(effects
@@
 		(property "Description" "Unpolarized capacitor, small symbol"
 			(at 116.84 93.98 0)
+			(effects
+				(font
+					(size 1.27 1.27)
+				)
+				(hide yes)
+			)
+		)
+		(property "Mouser Part Number" " 80-C0603C153K4RECTU "
+			(at 116.84 93.98 90)
 			(effects
 				(font
@@
 			)
 		)
-		(property "Footprint" ""
+		(property "Footprint" "Resistor_SMD:R_0603_1608Metric_Pad0.98x0.95mm_HandSolder"
 			(at 119.126 39.624 90)
 			(effects
@@
 		)
 		(property "Description" "Resistor, US symbol"
+			(at 118.11 39.37 0)
+			(effects
+				(font
+					(size 1.27 1.27)
+				)
+				(hide yes)
+			)
+		)
+		(property "Mouser Part Number" " 603-AC0603JR-131KL "
 			(at 118.11 39.37 0)
 			(effects
@@
 			)
 		)
-		(property "Footprint" ""
+		(property "Footprint" "Resistor_SMD:R_0603_1608Metric_Pad0.98x0.95mm_HandSolder"
 			(at 89.916 95.504 90)
 			(effects
@@
 		)
 		(property "Description" "Resistor, US symbol"
+			(at 88.9 95.25 0)
+			(effects
+				(font
+					(size 1.27 1.27)
+				)
+				(hide yes)
+			)
+		)
+		(property "Mouser Part Number" " 791-WR06X333JTL "
 			(at 88.9 95.25 0)
 			(effects
@@
 			)
 		)
-		(property "Footprint" ""
+		(property "Footprint" "Capacitor_SMD:C_0603_1608Metric_Pad1.08x0.95mm_HandSolder"
 			(at 119.0752 54.61 0)
 			(effects
@@
 		)
 		(property "Description" "Unpolarized capacitor"
+			(at 118.11 50.8 0)
+			(effects
+				(font
+					(size 1.27 1.27)
+				)
+				(hide yes)
+			)
+		)
+		(property "Mouser Part Number" " 810-CGA3E2X5R1A474MA "
 			(at 118.11 50.8 0)
 			(effects
@@
 		(unit 1)
 		(exclude_from_sim no)
-		(in_bom yes)
+		(in_bom no)
 		(on_board yes)
 		(dnp no)
@@
 			)
 		)
-		(property "Footprint" ""
+		(property "Footprint" "gbc_repro_lib:gbc_ir_leds"
 			(at 101.6 106.68 0)
 			(effects
@@
 		)
 		(property "Description" "NPN phototransistor, emitter/collector"
+			(at 106.68 109.22 0)
+			(effects
+				(font
+					(size 1.27 1.27)
+				)
+				(hide yes)
+			)
+		)
+		(property "Mouser Part Number" "~"
 			(at 106.68 109.22 0)
 			(effects
@@
 			)
 		)
-		(property "Footprint" ""
+		(property "Footprint" "Resistor_SMD:R_0603_1608Metric_Pad0.98x0.95mm_HandSolder"
 			(at 89.916 103.124 90)
 			(effects
@@
 			)
 		)
+		(property "Mouser Part Number" " 791-WR06X333JTL "
+			(at 88.9 102.87 0)
+			(effects
+				(font
+					(size 1.27 1.27)
+				)
+				(hide yes)
+			)
+		)
 		(pin "1"
 		)
@@
 		(unit 1)
 		(exclude_from_sim no)
-		(in_bom yes)
+		(in_bom no)
 		(on_board yes)
 		(dnp no)
@@
 			)
 		)
-		(property "Footprint" ""
+		(property "Footprint" "gbc_repro_lib:gbc_ir_leds"
 			(at 133.35 39.37 0)
 			(effects
@@
 		(property "Sim.Pins" "1=K 2=A"
 			(at 133.35 39.37 0)
+			(effects
+				(font
+					(size 1.27 1.27)
+				)
+				(hide yes)
+			)
+		)
+		(property "Mouser Part Number" "~"
+			(at 133.35 39.37 90)
 			(effects
 				(font
@@
 			)
 		)
-		(property "Footprint" ""
+		(property "Footprint" "Resistor_SMD:R_0603_1608Metric_Pad0.98x0.95mm_HandSolder"
 			(at 105.156 90.424 90)
 			(effects
@@
 		)
 		(property "Description" "Resistor, US symbol"
+			(at 104.14 90.17 0)
+			(effects
+				(font
+					(size 1.27 1.27)
+				)
+				(hide yes)
+			)
+		)
+		(property "Mouser Part Number" " 603-RT0603DRE072KL "
 			(at 104.14 90.17 0)
 			(effects
@@
 			)
 		)
-		(property "Footprint" ""
+		(property "Footprint" "Resistor_SMD:R_0603_1608Metric_Pad0.98x0.95mm_HandSolder"
 			(at 135.636 105.664 90)
 			(effects
@@
 		)
 		(property "Description" "Resistor, US symbol"
+			(at 134.62 105.41 0)
+			(effects
+				(font
+					(size 1.27 1.27)
+				)
+				(hide yes)
+			)
+		)
+		(property "Mouser Part Number" " 603-AC0603JR-07200KL "
 			(at 134.62 105.41 0)
 			(effects
@@
 			)
 		)
-		(property "Footprint" ""
+		(property "Footprint" "Capacitor_SMD:C_0603_1608Metric_Pad1.08x0.95mm_HandSolder"
 			(at 148.2852 109.22 0)
 			(effects
@@
 		)
 		(property "Description" "Unpolarized capacitor"
+			(at 147.32 105.41 0)
+			(effects
+				(font
+					(size 1.27 1.27)
+				)
+				(hide yes)
+			)
+		)
+		(property "Mouser Part Number" " 187-CL10C330JB8NNND "
 			(at 147.32 105.41 0)
 			(effects
@@
 			)
 		)
-		(property "Footprint" ""
+		(property "Footprint" "Resistor_SMD:R_0603_1608Metric_Pad0.98x0.95mm_HandSolder"
 			(at 119.126 32.004 90)
 			(effects
@@
 		)
 		(property "Description" "Resistor, US symbol"
+			(at 118.11 31.75 0)
+			(effects
+				(font
+					(size 1.27 1.27)
+				)
+				(hide yes)
+			)
+		)
+		(property "Mouser Part Number" " 708-RMCF0603JT150R "
 			(at 118.11 31.75 0)
 			(effects
@@
 			)
 		)
-		(property "Footprint" ""
+		(property "Footprint" "Resistor_SMD:R_0603_1608Metric_Pad0.98x0.95mm_HandSolder"
 			(at 129.286 90.424 90)
 			(effects
@@
 			(at 128.27 90.17 0)
 			(effects
+				(font
+					(size 1.27 1.27)
+				)
+				(hide yes)
+			)
+		)
+		(property "Mouser Part Number" " 279-CRG0603F1M0 "
+			(at 128.27 90.17 0)
+			(effects
