File: PCB/opengbc-pcb/pwr.kicad_sch (KiCad schematic)
At the start: 19 parts, among them J1 Barrel_Jack_Switch, U5 PWR_SWITCH, U6 Regulator board, U7 LD1117S33TR_SOT223

Commit message: :eyes:
Parts:
- removed BT1: 2xAA 3V, symbol Device:Battery
- removed FB6, FB7, FB8: FerriteBead_Small, symbol Device:FerriteBead_Small
- removed L1: L_Ferrite_Coupled, symbol Device:L_Ferrite_Coupled
- removed U5: PWR_SWITCH, symbol gbc_switch:PWR_SWITCH
- added D3: LED, LED_THT:LED_D3.0mm, symbol Device:LED
- added D4: 1SS355, Diode_SMD:D_SOD-323_HandSoldering, symbol Device:D
- added L1: Choke_CommonMode_FerriteCore_1243, Inductor_SMD:L_CommonModeChoke_Coilcraft_1812CAN, symbol Filter:Choke_CommonMode_FerriteCore_1243
- added Q4: 2SC4081UB, Package_TO_SOT_SMD:SOT-323_SC-70, symbol Transistor_BJT:Q_NPN_BEC
- added R20: 750R, Resistor_SMD:R_0603_1608Metric_Pad0.98x0.95mm_HandSolder, symbol Device:R_US
- added R21: 47k, Resistor_SMD:R_0603_1608Metric_Pad0.98x0.95mm_HandSolder, symbol Device:R_US
- added SW1: PWR_SWITCH, gbc_repro_lib:gbc_PowerSwitch, symbol gbc_switch:PWR_SWITCH
- C21: footprint (none) -> Capacitor_SMD:C_0603_1608Metric_Pad1.08x0.95mm_HandSolder; Mouser Part Number (none) -> 187-CL10A475KP8NNNC
- C22: footprint (none) -> Capacitor_SMD:CP_Elec_5x5.3; Mouser Part Number (none) -> 710-865080142007
- C23: footprint (none) -> Capacitor_SMD:C_0603_1608Metric_Pad1.08x0.95mm_HandSolder; Mouser Part Number (none) -> 81-GRM033R61C104KE4D
- C24: footprint (none) -> Capacitor_SMD:C_0603_1608Metric_Pad1.08x0.95mm_HandSolder; Mouser Part Number (none) -> 187-CL10A106KP8NNNC
- C7, C8: value .1uF -> 0.1uF; footprint (none) -> Capacitor_SMD:C_0603_1608Metric_Pad1.08x0.95mm_HandSolder; Mouser Part Number (none) -> 81-GRM033R61C104KE4D
- D2: footprint (none) -> Diode_SMD:D_SOD-323_HandSoldering; Mouser Part Number (none) -> 755-1SS355VMTE-17
- F1, F2: footprint (none) -> Fuse:Fuse_0603_1608Metric_Pad1.05x0.95mm_HandSolder; Mouser Part Number (none) -> 594-MFU0603FF01000P1
- P4: renamed from J1; footprint (none) -> gbc_repro_lib:SWITCHCRAFT_RAPC752SX; symbol Connector:Barrel_Jack_Switch -> gbc_dcjack:Barrel_Jack_Switch_MountingPin; Mouser Part Number (none) -> 502-RAPC752SX
- R19: footprint (none) -> Resistor_SMD:R_0603_1608Metric_Pad0.98x0.95mm_HandSolder; Mouser Part Number (none) -> 708-RMCF0603FT750R
- U6: footprint (none) -> gbc_repro_lib:GBC-PWRBD; now left out of the parts list
- U7: Mouser Part Number (none) -> 511-LD1117S33
Connections:
- net +5V: now also R21.1
- net GND: now also D4.1 (K), L1.2, SW1.MP
- net VCC: now also R20.1, SW1.C
- net at R19.1: now also SW1.1
- net at F1.2: now also SW1.3
- net B+: now reaches D2.1 (K), F1.1
- net B+: now also F2.2
- net at P4.1: now also L1.1
- net B-: now reaches P4.2
- net at P4.3: now also L1.4
- net at F2.1: now also L1.3
- new net: D3.1 (K), D4.2 (A)
- new net: D3.2 (A), Q4.2 (E)
- new net: Q4.1 (B), R21.2
- new net: Q4.3 (C), R20.2
- no-connect marks 2 -> 3
Other:
- moved on the sheet: F2
